File: AVRProgrammer.brd (EAGLE design)
At the start: 74.6 x 27.9 mm, 58 parts, among them Q1 SI1016CX-T1-GE3SOT-563F, U1 ESDS314, U10 SN74LVC1T45DRL, U11 SN74LVC1T45DRL, U2 XR22404SSOP28, U3 FT230XSSOP16, U4 ATmega88P-20AU A32, U6 CD4572UB, U7 SN74LVC2T45-Q1VSSOP-8, U8 SN74LVC1T45DRL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

Commit message: Replace incorrect USB ESD component
Parts:
- U1: value ESDS314 -> D5V0F4U6SO; device pepin:SOT95P282X145-5 -> pepin:SOT95P280X145-6
- moved U1 0.18 mm to (5.59, 22.1)
Connections:
- net N$32: now also U1.4; no longer U1.5
- net N$33: now also U1.3; no longer U1.4
- net N$34: now also U1.5; no longer U1.3
Routing:
- net N$32: track 32.1 -> 26.5 mm, vias 2 -> 3
- net GND: track 364.0 -> 359.9 mm
- net N$34: track 41.0 -> 43.9 mm, vias 3 -> 4
- net N$33: track 15.0 -> 17.8 mm
